File: rehabsense-main/rehabsense-main/haptic.kicad_sch (KiCad schematic)
At the start: 0 parts

Commit message: Adding schematics
Parts:
- added C10, C11, C12, C7, C8, C9: 1uF, symbol Device:C
- added C5: 10uF, symbol Device:C
- added C6: 0.1uF, symbol Device:C
- added U4, U5, U6: DRV2605LDGST, DRV2605LDGST:SOP50P490X110-10N, symbol DRV2605LDGST:DRV2605LDGST
Connections:
- new net: C9.1, U5.1 (REG)
- new net: C8.1, U4.1 (REG)
- new net: C11.1, U6.1 (REG)
- new net +3V3: C10.1, C12.1, C5.1, C6.1, C7.1, U4.10 (VDD), U4.5 (EN), U5.10 (VDD), U5.5 (EN), U6.10 (VDD), U6.5 (EN)
- new net DGND: C10.2, C11.2, C12.2, C5.2, C6.2, C7.2, C8.2, C9.2, U4.8 (GND), U5.8 (GND), U6.8 (GND)
- new net MOT1+: U4.7 (OUT+)
- new net MOT1-: U4.9 (OUT-)
- new net MOT2+: U5.7 (OUT+)
- new net MOT2-: U5.9 (OUT-)
- new net MOT3+: U6.7 (OUT+)
- new net MOT3-: U6.9 (OUT-)
- new net PWM1: U4.4 (IN/TRIG)
- new net PWM2: U5.4 (IN/TRIG)
- new net PWM3: U6.4 (IN/TRIG)
- new net SCL: U4.2 (SCL), U5.2 (SCL), U6.2 (SCL)
- new net SDA: U4.3 (SDA), U5.3 (SDA), U6.3 (SDA)
Other:
- note added: "Haptic Driver 1"
- note added: "Haptic Driver 2"
- note added: "Haptic Driver 3"
