File: rehabsense-main/rehabsense-main/mcu.kicad_sch (KiCad schematic)
At the start: 0 parts

Commit message: Adding schematics
Parts:
- added R3, R4: 2.2k, symbol Device:R
- added U3: XIAO_ESP32C3, XIAO_ESP32C3:MODULE_XIAO_ESP32C3, symbol XIAO_ESP32C3:XIAO_ESP32C3
Connections:
- new net +3V3: R3.1, R4.1
- new net DGND: U3.13 (GND)
- new net SCL: R4.2, U3.6 (D5)
- new net SDA: R3.2, U3.5 (D4)
