File: rehabsense-main/rehabsense-main/mcu.kicad_sch (KiCad schematic)
At the start: 3 parts, among them U3 XIAO_ESP32C3

Commit message: adding more circuits
Changed lines of the file:
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@@
+		)
+	)
+	(global_label "ADC2"
+		(shape input)
+		(at 151.13 87.63 0)
+		(fields_autoplaced yes)
+		(effects
+			(font
+				(size 1.27 1.27)
+			)
+			(justify left)
+		)
+		(property "Intersheetrefs" "${INTERSHEET_REFS}"
+			(at 158.9533 87.63 0)
+			(hide yes)
+			(show_name no)
+			(do_not_autoplace no)
+			(effects
+				(font
+					(size 1.27 1.27)
+				)
+				(justify left)
+			)
 		)
 	)
