File: rehabsense-main/rehabsense-main/adc.kicad_sch (KiCad schematic)
At the start: 4 parts, among them U10 LTC6903CMS8-TRPBF, U9 ADS131M02IPWR

Commit message: adding more circuits
Parts:
- added R31, R32: 4.7k, symbol Device:R
- R30: value R -> 4.7k
Connections:
- net +3V3A: now also U9.1 (AVDD)
- net AGND: now also U9.2 (AGND)
- net CLKIN: now also U9.17 (CLKIN)
- net MOSI: now also U9.16 (DIN)
- net SCK: now also U9.14 (SCLK)
- net RST: now reaches U9.11 (*SYNC/*RESET)
- net RST: now also R31.2
- net CS1: now reaches U9.12 (*CS)
- net CS1: now also R30.2
- net DRDY: now reaches U9.13 (*DRDY)
- net DRDY: now also R32.2
- net MISO: now reaches U9.15 (DOUT)
- net CAP: now reaches U9.18 (CAP)
- net DGND: now reaches U9.19 (DGND)
- net +3V3: now reaches U9.20 (DVDD)
- net +3V3: now also R30.1, R31.1, R32.1
- net AIN0+: now reaches U9.3 (AIN0P)
- net AIN0-: now reaches U9.4 (AIN0N)
- net AIN1-: now reaches U9.5 (AIN1N)
- net AIN1+: now reaches U9.6 (AIN1P)
Other:
- moved on the sheet: U9
