File: rehabsense-main/rehabsense-main/imu.kicad_sch (KiCad schematic)
At the start: 4 parts, among them U1 BMI270

Commit message: Adding schematics
Parts:
- added C3, C4: 0.1uF, symbol Device:C
- added R2: 100k, symbol Device:R
- added U2: BMI270, BMI270 (1):XDCR_BMI270, symbol BMI270:BMI270
Connections:
- net +3V3: now also C3.1, C4.1, R2.2, U2.5 (VDDIO), U2.8 (VDD)
- net DGND: now also C3.2, C4.2, U2.6 (GNDIO), U2.7 (GND)
- net SCL: now also U2.13 (SCX)
- net SDA: now also U2.14 (SDX)
- new net: R2.1, U2.1 (SDO)
Other:
- note added: "Bicep IMU I2C Address 0x69"
- note added: "Forearm IMU I2C Address 0x68"
- note added: "SPI"
- moved on the sheet: C1, C2, R1, U1

Commit message: adding more circuits
Connections:
- net CS_IMU1: now reaches U1.12 (CSB)
- net CS_IMU2: now reaches U2.12 (CSB)
Changed lines of the file:
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@@
+	(wire
+		(pts
+			(xy 71.12 81.28) (xy 76.2 81.28)
+		)
+		(stroke
+			(width 0)
+			(type default)
+		)
+	)
 	(wire
 		(pts
@@
 		(pts
 			(xy 69.85 91.44) (xy 76.2 91.44)
+		)
+		(stroke
+			(width 0)
+			(type default)
+		)
+	)
+	(wire
+		(pts
+			(xy 172.72 81.28) (xy 177.8 81.28)
 		)
 		(stroke
@@
 		)
 	)
+	(label "CS_IMU1"
+		(at 71.12 81.28 0)
+		(effects
+			(font
+				(size 1.27 1.27)
+			)
+			(justify bottom)
+		)
+	)
 	(label "SCL"
 		(at 71.12 86.36 0)
@@
 		)
 	)
+	(label "CS_IMU2"
+		(at 172.72 81.28 0)
+		(effects
+			(font
+				(size 1.27 1.27)
+			)
+			(justify bottom)
+		)
+	)
