File: final/schematics/emg.kicad_sch (KiCad schematic)
At the start: 42 parts, among them U7 TL074, U8 TL074

Commit message: fixing issues
Parts:
- removed U7, U8: TL074, symbol Amplifier_Operational:TL074
- added U7, U8: TL074HIPWR, TL074HIPWR:SOP65P640X120-14N, symbol TL074HIPWR:TL074HIPWR
- C13, C14, C15, C16, C17, C18, C19, C20, C21, C22, C23, C24: footprint (none) -> Capacitor_SMD:C_0603_1608Metric
- JP1, JP3: footprint (none) -> Jumper:SolderJumper-2_P1.3mm_Open_RoundedPad1.0x1.5mm
- JP2, JP4: footprint (none) -> Jumper:SolderJumper-3_P1.3mm_Open_RoundedPad1.0x1.5mm
- R10, R11, R12, R13, R14, R15, R16, R17, R18, R19, R20, R21, R22, R23, R24, R25, R26, R27, R28, R5, R6, R7, R8, R9: footprint (none) -> Resistor_SMD:R_0603_1608Metric
Connections:
- net ADC2: now also U8.8 (3OUT)
- net AGND: now also U7.11 (VCC-), U8.11 (VCC-)
- net IN+: now also U7.3 (1IN+), U8.3 (1IN+)
- net IN-: now also U7.5 (2IN+), U8.5 (2IN+)
- net A12: now reaches C18.2, R12.1, R13.2
- net A12: now also U7.12 (4IN+)
- net B1: now reaches R18.2, R21.1
- net B1: now also U8.1 (1OUT)
- net B2: now reaches R17.2, R18.1
- net B2: now also U8.2 (1IN-)
- net A6: now reaches R7.2, R8.1
- net A6: now also U7.6 (2IN-)
- net B6: now reaches R21.2, R22.1
- net B6: now also U8.6 (2IN-)
- net A2: now reaches R5.2, R6.1
- net A2: now also U7.2 (1IN-)
- net B12: now reaches C19.2, R19.1, R20.2
- net B12: now also U8.12 (4IN+)
- net A1: now reaches R6.2, R7.1
- net A1: now also U7.1 (1OUT)
- net +3V3A renamed +5
- net +5: now also U7.4 (VCC+), U8.4 (VCC+)
- net ampref1 renamed A13
- net A13: now also U7.13 (4IN-), U7.14 (4OUT)
- net ampref2 renamed B10
- net B10: now also U8.10 (3IN+), U8.13 (4IN-), U8.14 (4OUT)
- net bpfIN1 renamed 9
- net bpfIN2 renamed B9
- net B9: now also U8.9 (3IN-)
- net inaOUT1 renamed A7
- net A7: now also U7.7 (2OUT)
- net inaOUT2 renamed B7
- net B7: now also U8.7 (2OUT)
- new net A10: U7.10 (3IN+)
- new net A8: U7.8 (3OUT)
- new net A9: U7.9 (3IN-)
Other:
- note added: "TL074"
- moved on the sheet: JP2, JP4, R15, R16, R27, R28

Commit message: finishing
Connections:
- net +5 renamed +5VA

Commit message: finished
Parts:
- added J2, J3: SJ3-35083C-TR, SJ3-35083C-TR:SAMESKY_SJ3-35083C-TR, symbol SJ3-35083C-TR:SJ3-35083C-TR
Connections:
- net DRL renamed DRL1
- net DRL1: now also J2.1; no longer JP4.2 (C), R23.2
- net IN+ renamed IN1+
- net IN1+: now also J2.2; no longer C20.1, R28.2, U8.3 (1IN+)
- net IN- renamed IN1-
- net IN1-: now also J2.4; no longer C20.2, R27.1, U8.5 (2IN+)
- new net DRL2: J3.1, JP4.2 (C), R23.2
- new net IN2+: C20.1, J3.2, R28.2, U8.3 (1IN+)
- new net IN2-: C20.2, J3.4, R27.1, U8.5 (2IN+)
