File: final/schematics/rehabsense-main.kicad_pcb (KiCad board)
At the start: 2 copper layers, 74 parts, among them J1 B2B-PH-K-S, U1 BMI270, U10 LTC6903CMS8-TRPBF, U11 MP2161GJ-Z, U12 LT3045EMSE_PBF, U13 LTC3122EMSE_PBF, U2 BMI270, U3 XIAO_ESP32C3, U4 DRV2605LDGST, U5 DRV2605LDGST, U6 DRV2605LDGST, U7 TL074HIPWR, U8 TL074HIPWR, U9 ADS131M02IPWR

Commit message: finishing
Parts:
- added C25: 4.7uF 6.3V, Capacitor_SMD:C_1206_3216Metric, F.Cu at (149.8, 95.9)
- added C26: 4.7uF 6.3V, Capacitor_SMD:C_0603_1608Metric, F.Cu at (145.0, 90.8)
- added C27: 4.7uF, Capacitor_SMD:C_0603_1608Metric, F.Cu at (145.0, 93.3)
- added C28: 47uF 10V, Capacitor_SMD:C_1206_3216Metric, F.Cu at (149.8, 99.3)
- added C29: 150pF, Capacitor_SMD:C_0603_1608Metric, F.Cu at (145.0, 95.8)
- added C30: 12pF, Capacitor_SMD:C_0603_1608Metric, F.Cu at (145.0, 98.3)
- added C31: 10uF 10V, Capacitor_SMD:C_1206_3216Metric, F.Cu at (152.3, 107.7)
- added L2: 1uH ASMPM-0806-1R0M-T, ASMPM_0806_1R0M_T:INDC2016X100N, F.Cu at (149.2, 102.6)
- added L3: 1uH ASMPM-0806-1R0M-T, ASMPM_0806_1R0M_T:INDC2016X100N, F.Cu at (151.7, 111.0)
- added R33: 17.4k, Resistor_SMD:R_0603_1608Metric, F.Cu at (145.0, 100.8)
- added R34: 487k, Resistor_SMD:R_0603_1608Metric, F.Cu at (145.0, 103.3)
- added R35: 121k, Resistor_SMD:R_0603_1608Metric, F.Cu at (145.0, 105.8)
- added R36: 137k, Resistor_SMD:R_0603_1608Metric, F.Cu at (145.0, 108.3)
- added U14: LT3042EMSE-TRPBF, LT3042EMSE_TRPBF:05-08-1664_ADI, F.Cu at (150.7, 91.9)
Connections:
- net +5 renamed +5VA
- J1 pad 1: /power/VBAT+ -> +BATT
- J1 pad 2: unconnected-(J1-Pad2) -> DGND
- U11 pad 1: unconnected-(U11-PG-Pad1) -> /power/PG
- U11 pad 2: unconnected-(U11-VIN-Pad2) -> +6VD
- U11 pad 3: unconnected-(U11-SW-Pad3) -> Net-(U11-SW)
- U11 pad 5: unconnected-(U11-OUT-Pad5) -> Net-(U11-OUT)
- U13 pad 1: unconnected-(U13-SW-Pad1) -> Net-(U13-SW)
- U13 pad 10: unconnected-(U13-SGND-Pad10) -> DGND
- U13 pad 11: unconnected-(U13-VOUT-Pad11) -> Net-(U13-VOUT)
- U13 pad 12: unconnected-(U13-CAP-Pad12) -> Net-(U13-CAP)
- U13 pad 13: unconnected-(U13-EPAD-Pad13) -> DGND
- U13 pad 2: unconnected-(U13-PGND-Pad2) -> DGND
- U13 pad 3: unconnected-(U13-VIN-Pad3) -> +BATT
- U13 pad 4: unconnected-(U13-PWM/SYNC-Pad4) -> Net-(U13-PWM/SYNC)
- U13 pad 5: unconnected-(U13-VCC-Pad5) -> Net-(U13-PWM/SYNC)
- U13 pad 6: unconnected-(U13-RT-Pad6) -> Net-(U13-RT)
- U13 pad 7: unconnected-(U13-VC-Pad7) -> Net-(U13-VC)
- U13 pad 8: unconnected-(U13-FB-Pad8) -> Net-(U13-FB)

Commit message: fixed layout
Parts:
- added C32: 10uF 10V, Capacitor_SMD:C_1206_3216Metric, F.Cu at (161.8, 84.7)
- added C33: 4.7uF 10V, Capacitor_SMD:C_1206_3216Metric, F.Cu at (161.8, 88.0)
- added C34: 470nF 10V, Capacitor_SMD:C_1206_3216Metric, F.Cu at (161.8, 91.4)
- added C35: 10uF 6.3V, Capacitor_SMD:C_1206_3216Metric, F.Cu at (161.8, 94.7)
- added C36: 10uF 10V, Capacitor_SMD:C_1206_3216Metric, F.Cu at (161.8, 98.1)
- added C37: 470nF 10V, Capacitor_SMD:C_1206_3216Metric, F.Cu at (161.8, 101.4)
- added C38: 4.7uF 10V, Capacitor_SMD:C_1206_3216Metric, F.Cu at (161.8, 104.8)
- added C39: 10uF, Capacitor_SMD:C_0603_1608Metric, F.Cu at (176.7, 84.3)
- added C40: 0.1uF, Capacitor_SMD:C_0603_1608Metric, F.Cu at (176.7, 86.8)
- added C41: 10uF, Capacitor_SMD:C_0603_1608Metric, F.Cu at (176.7, 89.3)
- added C42: 0.1uF, Capacitor_SMD:C_0603_1608Metric, F.Cu at (176.7, 91.8)
- added C43: 1uF, Capacitor_SMD:C_0603_1608Metric, F.Cu at (176.7, 96.3)
- added C44: 0.1uF, Capacitor_SMD:C_0603_1608Metric, F.Cu at (176.7, 98.8)
- added C45: 1uF, Capacitor_SMD:C_0603_1608Metric, F.Cu at (176.7, 101.3)
- added C46: 0.1uF, Capacitor_SMD:C_0603_1608Metric, F.Cu at (176.7, 103.8)
- added C47: 1uF, Capacitor_SMD:C_0603_1608Metric, F.Cu at (176.7, 106.3)
- added C48: 0.1uF, Capacitor_SMD:C_0603_1608Metric, F.Cu at (176.7, 108.8)
- added R37: 200k, Resistor_SMD:R_0603_1608Metric, F.Cu at (166.7, 84.3)
- added R38: 44.2k, Resistor_SMD:R_0603_1608Metric, F.Cu at (166.7, 86.8)
- added R39: 33.2k, Resistor_SMD:R_0603_1608Metric, F.Cu at (166.7, 89.3)
- added R41: 49.9k, Resistor_SMD:R_0603_1608Metric, F.Cu at (166.7, 91.8)
- added U14: LT3045EMSE_PBF, LT3045EMSE_PBF:SOP65P490X110-13N, F.Cu at (169.0, 95.8)
Connections:
- net /adc/CS2 renamed CS
- net /adc/MISO renamed MISO
- net /adc/MOSI renamed MOSI
- net /adc/SCK renamed SCK
- C27 pad 2: Net-(U13-VOUT) -> +6VD
- C28 pad 2: Net-(U13-VOUT) -> +6VD
- C31 pad 1: unconnected-(C31-Pad1) -> DGND
- C5 pad 1: +3V3 -> +3V3D
- C6 pad 1: +3V3 -> +3V3D
- L3 pad 2: Net-(U11-OUT) -> +3V3D
- R29 pad 1: +3V3A -> +3V3D
- R30 pad 1: +3V3 -> +3V3D
- R31 pad 1: +3V3 -> +3V3D
- R32 pad 1: +3V3 -> +3V3D
- R34 pad 1: Net-(U13-VOUT) -> +6VD
- U10 pad 7: +3V3A -> +3V3D
- U10 pad 8: +3V3A -> +3V3D
- U11 pad 4: unconnected-(U11-PGND-Pad4) -> DGND
- U11 pad 5: Net-(U11-OUT) -> +3V3D
- U11 pad 6: unconnected-(U11-AGND-Pad6) -> DGND
- U11 pad 7: unconnected-(U11-FB-Pad7) -> Net-(U11-FB)
- U11 pad 8: unconnected-(U11-EN-Pad8) -> /power/EN_DIG
- U12 pad 1: unconnected-(U12-IN-Pad1) -> +5VA
- U12 pad 10: unconnected-(U12-OUTS-Pad10) -> +3V3A
- U12 pad 11: unconnected-(U12-OUT-Pad11) -> +3V3A
- U12 pad 12: unconnected-(U12-OUT__1-Pad12) -> +3V3A
- U12 pad 13: unconnected-(U12-EXP-Pad13) -> AGND
- U12 pad 2: unconnected-(U12-IN__1-Pad2) -> +5VA
- U12 pad 3: unconnected-(U12-IN__2-Pad3) -> +5VA
- U12 pad 4: unconnected-(U12-EN/UV-Pad4) -> +5VA
- U12 pad 6: unconnected-(U12-ILIM-Pad6) -> AGND
- U12 pad 7: unconnected-(U12-PGFB-Pad7) -> +5VA
- U12 pad 8: unconnected-(U12-SET-Pad8) -> Net-(U12-SET)
- U12 pad 9: unconnected-(U12-GND-Pad9) -> AGND
- U13 pad 11: Net-(U13-VOUT) -> +6VD
- U9 pad 20: +3V3 -> +3V3D
- U9 pad 3: /adc/AIN0+ -> ADC1
- U9 pad 4: /adc/AIN0- -> AGND
- U9 pad 5: /adc/AIN1- -> AGND
- U9 pad 6: /adc/AIN1+ -> ADC2

Commit message: finished
Parts:
- removed C11, C12: 1uF, Capacitor_SMD:C_0603_1608Metric
- removed C41: 10uF, Capacitor_SMD:C_0603_1608Metric
- removed C42: 0.1uF, Capacitor_SMD:C_0603_1608Metric
- removed the U14 at (169.0, 95.8)
- removed the U14 at (150.7, 91.9)
- added J2: SJ3-35083C-TR, SJ3-35083C-TR:SAMESKY_SJ3-35083C-TR, F.Cu at (143.0, 69.3)
- added J3: SJ3-35083C-TR, SJ3-35083C-TR:SAMESKY_SJ3-35083C-TR, F.Cu at (153.3, 69.3)
- added JP5: SolderJumper_2_Open, Jumper:SolderJumper-2_P1.3mm_Open_RoundedPad1.0x1.5mm, F.Cu at (176.4, 119.5)
- added JP6: SolderJumper_2_Open, Jumper:SolderJumper-2_P1.3mm_Open_RoundedPad1.0x1.5mm, F.Cu at (176.4, 123.1)
- added L1: MPZ1608S601ATA00, MPZ1608S601ATA00 (1):INDC1608X95N, F.Cu at (144.9, 107.1)
- added R40: RC0603JR-070RL, RC0603JR-070RL:RC0603N_YAG, F.Cu at (144.9, 109.6)
- added R42: 2.2k, Resistor_SMD:R_0603_1608Metric, F.Cu at (161.0, 100.9)
- added R43: 2.2k, Resistor_SMD:R_0603_1608Metric, F.Cu at (161.0, 103.4)
- added R44: 2.2k, Resistor_SMD:R_0603_1608Metric, F.Cu at (161.0, 105.9)
- added R45: 2.2k, Resistor_SMD:R_0603_1608Metric, F.Cu at (161.0, 108.5)
- added R46: 10k, Resistor_SMD:R_0603_1608Metric, F.Cu at (165.0, 95.9)
- added R47: 10k, Resistor_SMD:R_0603_1608Metric, F.Cu at (165.0, 98.4)
- added R48: 10k, Resistor_SMD:R_0603_1608Metric, F.Cu at (165.0, 100.9)
- added TP1: TestPoint, Connector_Pin:Pin_D1.0mm_L10.0mm_LooseFit, F.Cu at (130.9, 96.9)
- added TP10: TestPoint, Connector_Pin:Pin_D1.0mm_L10.0mm_LooseFit, F.Cu at (183.8, 72.1)
- added TP11: TestPoint, Connector_Pin:Pin_D1.0mm_L10.0mm_LooseFit, F.Cu at (188.2, 63.2)
- added TP12: TestPoint, Connector_Pin:Pin_D1.0mm_L10.0mm_LooseFit, F.Cu at (188.2, 67.7)
- added TP13: TestPoint, Connector_Pin:Pin_D1.0mm_L10.0mm_LooseFit, F.Cu at (188.2, 72.1)
- added TP14: TestPoint, Connector_Pin:Pin_D1.0mm_L10.0mm_LooseFit, F.Cu at (192.7, 63.2)
- added TP15: TestPoint, Connector_Pin:Pin_D1.0mm_L10.0mm_LooseFit, F.Cu at (192.7, 67.7)
- added TP16: TestPoint, Connector_Pin:Pin_D1.0mm_L10.0mm_LooseFit, F.Cu at (192.7, 72.1)
- added TP17: TestPoint, Connector_Pin:Pin_D1.0mm_L10.0mm_LooseFit, F.Cu at (169.2, 96.9)
- added TP18: TestPoint, Connector_Pin:Pin_D1.0mm_L10.0mm_LooseFit, F.Cu at (169.2, 101.3)
- added TP19: MOT1+, Connector_Pin:Pin_D1.1mm_L8.5mm_W2.5mm_FlatFork, F.Cu at (152.6, 97.0)
- added TP2: TestPoint, Connector_Pin:Pin_D1.0mm_L10.0mm_LooseFit, F.Cu at (130.9, 101.3)
- added TP20: MOT1-, Connector_Pin:Pin_D1.1mm_L8.5mm_W2.5mm_FlatFork, F.Cu at (152.6, 101.6)
- added TP21: MOT2+, Connector_Pin:Pin_D1.1mm_L8.5mm_W2.5mm_FlatFork, F.Cu at (152.6, 106.3)
- added TP22: MOT2-, Connector_Pin:Pin_D1.1mm_L8.5mm_W2.5mm_FlatFork, F.Cu at (152.6, 110.9)
- added TP3: TestPoint, Connector_Pin:Pin_D1.0mm_L10.0mm_LooseFit, F.Cu at (130.9, 105.8)
- added TP4: TestPoint, Connector_Pin:Pin_D1.0mm_L10.0mm_LooseFit, F.Cu at (130.9, 110.2)
- added TP5: TestPoint, Connector_Pin:Pin_D1.0mm_L10.0mm_LooseFit, F.Cu at (135.3, 96.9)
- added TP6: TestPoint, Connector_Pin:Pin_D1.0mm_L10.0mm_LooseFit, F.Cu at (135.3, 101.3)
- added TP7: TestPoint, Connector_Pin:Pin_D1.0mm_L10.0mm_LooseFit, F.Cu at (135.3, 105.8)
- added TP8: TestPoint, Connector_Pin:Pin_D1.0mm_L10.0mm_LooseFit, F.Cu at (183.8, 63.2)
- added TP9: TestPoint, Connector_Pin:Pin_D1.0mm_L10.0mm_LooseFit, F.Cu at (183.8, 67.7)
- added U14: LT3045EMSE_PBF, LT3045EMSE_PBF:SOP65P490X110-13N, F.Cu at (141.9, 103.0)
- U3: value XIAO_ESP32C3 -> TCA9543APWR; footprint XIAO_ESP32C3:MODULE_XIAO_ESP32C3 -> TCA9543APWR:IC_TCA9543APWR
- U6: value DRV2605LDGST -> XIAO_ESP32_S3; footprint DRV2605LDGST:SOP50P490X110-10N -> XIAO_ESP32_S3:MODULE_XIAO_ESP32_S3
- moved R4 67.3 mm to (183.5, 78.1)
- moved R3 67.3 mm to (183.5, 75.6)
- moved U9 56.6 mm to (186.9, 98.8)
- moved U10 56.6 mm to (186.0, 105.3)
- moved C1 56.1 mm to (181.1, 110.9)
- moved C2 56.1 mm to (181.1, 113.4)
- moved C3 56.1 mm to (181.1, 115.9)
- moved C4 56.1 mm to (181.1, 118.4)
- moved R1 56.1 mm to (181.1, 121.0)
- moved R2 56.1 mm to (181.1, 123.5)
- moved R29 56.1 mm to (180.2, 98.4)
- moved R30 56.1 mm to (180.2, 100.9)
- moved R31 56.1 mm to (180.2, 103.4)
- moved R32 56.1 mm to (180.2, 105.9)
- moved U4 52.8 mm to (168.5, 112.0)
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Connections:
- net /haptic/MOT3+ renamed PWM_HAP1
- net /imu/CS_IMU2 renamed CS_IMU2
- C13 pad 1: IN+ -> IN1+
- C13 pad 2: IN- -> IN1-
- C20 pad 1: IN+ -> IN2+
- C20 pad 2: IN- -> IN2-
- JP2 pad 2: DRL -> DRL1
- JP4 pad 2: DRL -> DRL2
- R1 pad 1: Net-(U1-SDO) -> Net-(JP5-A)
- R14 pad 2: DRL -> DRL1
- R15 pad 1: IN- -> IN1-
- R16 pad 2: IN+ -> IN1+
- R2 pad 1: Net-(U2-SDO) -> Net-(JP6-A)
- R23 pad 2: DRL -> DRL2
- R27 pad 1: IN- -> IN2-
- R28 pad 2: IN+ -> IN2+
- R3 pad 2: /mcu/SDA -> SDA
- R4 pad 2: /mcu/SCL -> SCL
- U1 pad 1: Net-(U1-SDO) -> MISO
- U1 pad 12: /imu/CS_IMU1 -> CS_IMU1
- U1 pad 13: /imu/SCL -> SCK
- U1 pad 14: /imu/SDA -> MOSI
- U2 pad 1: Net-(U2-SDO) -> MISO
- U2 pad 13: /imu/SCL -> SCK
- U2 pad 14: /imu/SDA -> MOSI
- U3 pad 1: unconnected-(U3-D0-Pad1) -> DGND
- U3 pad 10: unconnected-(U3-D9-Pad10) -> Net-(U3-SC1)
- U3 pad 12: unconnected-(U3-VCC_3V3-Pad12) -> SCL
- U3 pad 13: DGND -> SDA
- U3 pad 14: unconnected-(U3-VUSB-Pad14) -> +3V3D
- U3 pad 2: unconnected-(U3-D1-Pad2) -> DGND
- U3 pad 3: unconnected-(U3-D2-Pad3) -> Net-(U3-~{RESET})
- U3 pad 4: unconnected-(U3-D3-Pad4) -> Net-(U3-~{INT0})
- U3 pad 5: /mcu/SDA -> Net-(U3-SD0)
- U3 pad 6: /mcu/SCL -> Net-(U3-SC0)
- U3 pad 7: unconnected-(U3-TX_D6-Pad7) -> DGND
- U3 pad 8: unconnected-(U3-RX_D7-Pad8) -> Net-(U3-~{INT1})
- U3 pad 9: unconnected-(U3-D8-Pad9) -> Net-(U3-SD1)
- U4 pad 2: /haptic/SCL -> SCL
- U4 pad 3: /haptic/SDA -> SDA
- U5 pad 2: /haptic/SCL -> SCL
- U5 pad 3: /haptic/SDA -> SDA
- U6 pad 1: Net-(U6-REG) -> CS_ADC
- U6 pad 10: +3V3D -> MISO
- U6 pad 2: /haptic/SCL -> DRDY_ADC
- U6 pad 3: /haptic/SDA -> CS_ADC
- U6 pad 4: /haptic/PWM3 -> CS_IMU1
- U6 pad 5: +3V3D -> SDA
- U6 pad 6: (no net) -> SCL
- U6 pad 8: DGND -> CS_IMU2/PWM_HAP2
- U6 pad 9: /haptic/MOT3- -> SCK
- U7 pad 3: IN+ -> IN1+
- U7 pad 5: IN- -> IN1-
- U8 pad 3: IN+ -> IN2+
- U8 pad 5: IN- -> IN2-
