File: final/schematics/imu.kicad_sch (KiCad schematic)
At the start: 8 parts, among them U1 BMI270, U2 BMI270

Commit message: fixing issues
Parts:
- C1, C2, C3, C4: footprint (none) -> Capacitor_SMD:C_0603_1608Metric
- R1, R2: footprint (none) -> Resistor_SMD:R_0603_1608Metric
Connections:
- net +3V3 renamed +3V3D
Changed lines of the file:
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@@
 		(in_pos_files yes)
 		(dnp no)
-		(fields_autoplaced yes)
 		(property "Reference" "#PWR07"
 			(at 212.09 72.39 0)
@@
 			)
 		)
-		(property "Value" "+3V3"
-			(at 212.09 63.5 0)
-			(show_name no)
-			(do_not_autoplace no)
-			(effects
-				(font
-					(size 1.27 1.27)
-				)
+		(property "Value" "+3V3D"
+			(at 208.534 64.516 0)
+			(show_name no)
+			(do_not_autoplace no)
+			(effects
+				(font
+					(size 1.27 1.27)
+				)
+				(justify left)
 			)
 		)
@@
 			)
 		)
-		(property "Footprint" ""
+		(property "Footprint" "Resistor_SMD:R_0603_1608Metric"
 			(at 68.072 96.52 90)
 			(hide yes)
@@
 			)
 		)
-		(property "Footprint" ""
+		(property "Footprint" "Capacitor_SMD:C_0603_1608Metric"
 			(at 230.8352 80.01 0)
 			(hide yes)
@@
 			)
 		)
-		(property "Footprint" ""
+		(property "Footprint" "Capacitor_SMD:C_0603_1608Metric"
 			(at 216.8652 80.01 0)
 			(hide yes)
@@
 		(in_pos_files yes)
 		(dnp no)
-		(fields_autoplaced yes)
 		(property "Reference" "#PWR09"
 			(at 166.37 85.09 0)
@@
 			)
 		)
-		(property "Value" "+3V3"
-			(at 166.37 76.2 0)
-			(show_name no)
-			(do_not_autoplace no)
-			(effects
-				(font
-					(size 1.27 1.27)
-				)
+		(property "Value" "+3V3D"
+			(at 162.56 76.708 0)
+			(show_name no)
+			(do_not_autoplace no)
+			(effects
+				(font
+					(size 1.27 1.27)
+				)
+				(justify left)
 			)
 		)
@@
 		(in_pos_files yes)
 		(dnp no)
-		(fields_autoplaced yes)
 		(property "Reference" "#PWR01"
 			(at 110.49 72.39 0)
@@
 			)
 		)
-		(property "Value" "+3V3"
-			(at 110.49 63.5 0)
-			(show_name no)
-			(do_not_autoplace no)
-			(effects
-				(font
-					(size 1.27 1.27)
-				)
+		(property "Value" "+3V3D"
+			(at 106.934 64.77 0)
+			(show_name no)
+			(do_not_autoplace no)
+			(effects
+				(font
+					(size 1.27 1.27)
+				)
+				(justify left)
 			)
 		)
@@
 			)
 		)
-		(property "Footprint" ""
+		(property "Footprint" "Capacitor_SMD:C_0603_1608Metric"
 			(at 115.2652 80.01 0)
 			(hide yes)
@@
 			)
 		)
-		(property "Footprint" ""
+		(property "Footprint" "Resistor_SMD:R_0603_1608Metric"
 			(at 168.148 86.36 90)
 			(hide yes)
@@
 			)
 		)
-		(property "Footprint" ""
+		(property "Footprint" "Capacitor_SMD:C_0603_1608Metric"
 			(at 129.2352 80.01 0)
 			(hide yes)

Commit message: finishing
Other:
- moved on the sheet: C3, C4, R2, U2

Commit message: finished
Parts:
- added JP5, JP6: SolderJumper_2_Open, Jumper:SolderJumper-2_P1.3mm_Open_RoundedPad1.0x1.5mm, symbol Jumper:SolderJumper_2_Open
Connections:
- net at R1.1: now also JP5.1 (A); no longer U1.1 (SDO)
- net at R2.1: now also JP6.1 (A); no longer U2.1 (SDO)
- net SCL renamed SCK
- net SDA renamed MOSI
- new net MISO: JP5.2 (B), JP6.2 (B), U1.1 (SDO), U2.1 (SDO)
Other:
- note added: "Forearm IMU SPI Mode, solder to activate I2C mode I2C Address 0x68"
- note added: "Forearm IMU SPI Mode, solder to activate I2C mode I2C Address 0x69"
- note removed: "Bicep IMU I2C Address 0x69"
- note removed: "Forearm IMU I2C Address 0x68"
- note removed: "SPI"
- moved on the sheet: R1, R2

Commit message: fixing
Parts:
- removed JP5, JP6: SolderJumper_2_Open, Jumper:SolderJumper-2_P1.3mm_Open_RoundedPad1.0x1.5mm, symbol Jumper:SolderJumper_2_Open
- added JP10, JP11, JP12, JP7, JP8, JP9: SolderJumper_3_Open, Jumper:SolderJumper-3_P1.3mm_Open_RoundedPad1.0x1.5mm, symbol Jumper:SolderJumper_3_Open
Connections:
- net MISO: now also JP12.3 (B), JP7.3 (B); no longer U1.1 (SDO), U2.1 (SDO)
- net MOSI: now also JP11.3 (B), JP8.3 (B); no longer U1.14 (SDX), U2.14 (SDX)
- net SCK: now also JP10.3 (B), JP9.3 (B); no longer U1.13 (SCX), U2.13 (SCX)
- net at R2.1: now also JP12.1 (A)
- net at R1.1: now also JP7.1 (A)
- new net: JP8.2 (C), U1.14 (SDX)
- new net: JP10.2 (C), U2.13 (SCX)
- new net: JP12.2 (C), U2.1 (SDO)
- new net: JP9.2 (C), U1.13 (SCX)
- new net: JP7.2 (C), U1.1 (SDO)
- new net: JP11.2 (C), U2.14 (SDX)
- new net SCL: JP10.1 (A), JP9.1 (A)
- new net SDA: JP11.1 (A), JP8.1 (A)
Other:
- moved on the sheet: C3, C4, R1, R2, U2
