File: final/schematics/mcu.kicad_sch (KiCad schematic)
At the start: 3 parts, among them U3 XIAO_ESP32C3

Commit message: fixing issues
Parts:
- R3, R4: footprint (none) -> Resistor_SMD:R_0603_1608Metric
Connections:
- net +3V3 renamed +3V3D
Changed lines of the file:
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@@
 			)
 		)
-		(property "Value" "+3V3"
-			(at 86.36 63.5 0)
+		(property "Value" "+3V3D"
+			(at 88.9 67.3099 0)
 			(show_name no)
 			(do_not_autoplace no)
@@
 					(size 1.27 1.27)
 				)
+				(justify left)
 			)
 		)
@@
 			)
 		)
-		(property "Footprint" ""
+		(property "Footprint" "Resistor_SMD:R_0603_1608Metric"
 			(at 92.202 74.93 90)
 			(hide yes)
@@
 			)
 		)
-		(property "Footprint" ""
+		(property "Footprint" "Resistor_SMD:R_0603_1608Metric"
 			(at 84.582 74.93 90)
 			(hide yes)

Commit message: finishing
Changed lines of the file:
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@@
 		)
 	)
-	(global_label "ADC2"
+	(global_label "MISO"
 		(shape input)
-		(at 151.13 87.63 0)
+		(at 158.75 73.66 0)
 		(fields_autoplaced yes)
 		(effects
@@
 		)
 		(property "Intersheetrefs" "${INTERSHEET_REFS}"
-			(at 158.9533 87.63 0)
+			(at 166.3314 73.66 0)
 			(hide yes)
 			(show_name no)
@@
 		)
 	)
-	(global_label "ADC1"
+	(global_label "MOSI"
 		(shape input)
-		(at 151.13 80.01 0)
+		(at 158.75 71.12 0)
 		(fields_autoplaced yes)
 		(effects
@@
 		)
 		(property "Intersheetrefs" "${INTERSHEET_REFS}"
-			(at 158.9533 80.01 0)
+			(at 166.3314 71.12 0)
 			(hide yes)
 			(show_name no)
+			(do_not_autoplace no)
+			(effects
+				(font
+					(size 1.27 1.27)
+				)
+				(justify left)
+			)
+		)
+	)
+	(global_label "SCK"
+		(shape input)
+		(at 158.75 76.2 0)
+		(fields_autoplaced yes)
+		(effects
+			(font
+				(size 1.27 1.27)
+			)
+			(justify left)
+		)
+		(property "Intersheetrefs" "${INTERSHEET_REFS}"
+			(at 165.4847 76.2 0)
+			(hide yes)
+			(show_name no)

Commit message: finished
Parts:
- removed U3: XIAO_ESP32C3, XIAO_ESP32C3:MODULE_XIAO_ESP32C3, symbol XIAO_ESP32C3:XIAO_ESP32C3
- added TP10, TP11, TP12, TP13, TP14, TP15, TP16, TP8, TP9: TestPoint, Connector_Pin:Pin_D1.0mm_L10.0mm_LooseFit, symbol Connector:TestPoint
- added U6: XIAO_ESP32_S3, XIAO_ESP32_S3:MODULE_XIAO_ESP32_S3, symbol XIAO_ESP32_S3:XIAO_ESP32_S3
Connections:
- net +3V3D: now also U6.12 (3V3)
- net DGND: now also U6.13 (GND)
- net MISO: now also TP9.1, U6.10 (D9/GPIO8)
- net MOSI: now also TP10.1, U6.11 (D10/GPIO9)
- net SCK: now also TP8.1, U6.9 (D8/GPIO7)
- net SCL: now also TP16.1, U6.6 (D5/GPIO6)
- net SDA: now also TP15.1, U6.5 (D4/GPIO5)
- new net CS_ADC: TP11.1, TP12.1, U6.1 (D0/GPIO1), U6.3 (D2/GPIO3)
- new net CS_IMU1: TP14.1, U6.4 (D3/GPIO4)
- new net CS_IMU2/PWM_HAP2: U6.8 (D7/GPIO44)
- new net DRDY_ADC: TP13.1, U6.2 (D1/GPIO2)
- new net PWM_HAP1: U6.7 (D6/GPIO43)
Other:
- moved on the sheet: R3, R4

Commit message: fixed jumper connection
Parts:
- added JP7: SolderJumper_3_Open, Jumper:SolderJumper-3_P1.3mm_Open_RoundedPad1.0x1.5mm, symbol Jumper:SolderJumper_3_Open
Connections:
- net CS_IMU2/PWM_HAP2: no longer names the net of U6.8 (D7/GPIO44)
- net CS_IMU2/PWM_HAP2: now also JP7.2 (C)
- new net CS_IMU2: JP7.1 (A)
- new net PWM_HAP2: JP7.3 (B)
Changed lines of the file:
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@@
 	(wire
 		(pts
-			(xy 149.86 73.66) (xy 156.21 73.66)
+			(xy 149.86 73.66) (xy 171.45 73.66)
 		)
 		(stroke
@@
 	(wire
 		(pts
+			(xy 175.26 66.04) (xy 175.26 68.58)
+		)
+		(stroke
+			(width 0)
+			(type default)
+		)
+	)
+	(wire
+		(pts
 			(xy 154.94 83.82) (xy 156.21 83.82)
 		)
@@
 	(wire
 		(pts
+			(xy 177.8 66.04) (xy 175.26 66.04)
+		)
+		(stroke
+			(width 0)
+			(type default)
+		)
+	)
+	(wire
+		(pts
 			(xy 86.36 71.12) (xy 86.36 69.85)
 		)
@@
 	(wire
 		(pts
+			(xy 177.8 81.28) (xy 175.26 81.28)
+		)
+		(stroke
+			(width 0)
+			(type default)
+		)
+	)
+	(wire
+		(pts
 			(xy 153.67 60.96) (xy 153.67 63.5)
 		)
@@
 		(pts
 			(xy 152.4 91.44) (xy 152.4 88.9)
+		)
+		(stroke
+			(width 0)
+			(type default)
+		)
+	)
+	(wire
+		(pts
+			(xy 175.26 81.28) (xy 175.26 78.74)
 		)
 		(stroke
@@
 		)
 	)
-	(global_label "CS_IMU2{slash}PWM_HAP2"
+	(global_label "CS_IMU2"
 		(shape input)
-		(at 156.21 73.66 0)
+		(at 177.8 66.04 0)
 		(fields_autoplaced yes)
 		(effects
@@
 		)
 		(property "Intersheetrefs" "${INTERSHEET_REFS}"
-			(at 178.608 73.66 0)
+			(at 188.8285 66.04 0)
 			(hide yes)
 			(show_name no)
@@
 				)
 				(justify right)
+			)
+		)
+	)
+	(global_label "PWM_HAP2"
+		(shape input)
+		(at 177.8 81.28 0)
+		(fields_autoplaced yes)
+		(effects
+			(font
+				(size 1.27 1.27)
+			)
+			(justify left)
+		)
+		(property "Intersheetrefs" "${INTERSHEET_REFS}"
+			(at 190.8242 81.28 0)
+			(hide yes)
+			(show_name no)
+			(do_not_autoplace no)
+			(effects
+				(font
+					(size 1.27 1.27)
+				)
+				(justify left)
 			)
 		)
@@
 					(unit 1)
 				)
+			)
+		)
+	)
+	(symbol
+		(lib_id "Jumper:SolderJumper_3_Open")
+		(at 175.26 73.66 270)
+		(unit 1)
+		(body_style 1)
+		(exclude_from_sim no)
+		(in_bom no)
+		(on_board yes)
+		(in_pos_files yes)
+		(dnp no)
+		(fields_autoplaced yes)
+		(property "Reference" "JP7"
+			(at 177.8 72.3899 90)
+			(show_name no)
+			(do_not_autoplace no)
+			(effects
+				(font
+					(size 1.27 1.27)
+				)
+				(justify left)
+			)
+		)
+		(property "Value" "SolderJumper_3_Open"
+			(at 177.8 74.9299 90)
+			(show_name no)
+			(do_not_autoplace no)
+			(effects
+				(font
+					(size 1.27 1.27)
+				)
+				(justify left)
+			)
+		)
+		(property "Footprint" "Jumper:SolderJumper-3_P1.3mm_Open_RoundedPad1.0x1.5mm"
+			(at 175.26 73.66 0)
+			(hide yes)
+			(show_name no)
+			(do_not_autoplace no)
+			(effects
+				(font
+					(size 1.27 1.27)
+				)
+			)
+		)
+		(property "Datasheet" ""
+			(at 160.02 73.66 0)
+			(hide yes)
+			(show_name no)
+			(do_not_autoplace no)
+			(effects
+				(font
+					(size 1.27 1.27)
+				)
+			)
+		)
+		(property "Description" "Solder Jumper, 3-pole, open"
+			(at 162.56 73.66 0)
+			(hide yes)
+			(show_name no)
+			(do_not_autoplace no)
+			(effects
+				(font
+					(size 1.27 1.27)
+				)
+			)
+		)
+		(property private "KLC_S5.1" "This is a generic symbol, it has fp-filter, but no default footprint"
+			(at 157.48 73.66 0)
+			(hide yes)
+			(show_name yes)
+			(do_not_autoplace no)
+			(effects
+				(font
+					(size 1.27 1.27)
+				)
+			)
+		)
+		(property private "KLC_S3.3" "Graphical-Symbol: thickness is 6mm, fill is background"
+			(at 154.94 73.66 0)
+			(hide yes)
+			(show_name yes)
+			(do_not_autoplace no)
+			(effects
+				(font
+					(size 1.27 1.27)
+				)
+			)
+		)
+		(pin "1"
+		)
+		(pin "2"
+		)
+		(pin "3"
+		)
+		(instances
+			(project "rehabsense-main"
+				(path "/b751250a-7d43-475a-8447-686d399cd67b/4c292b8e-bacf-4862-ad93-06ae5fddd327"
+					(reference "JP7")
+					(unit 1)
+				)

Commit message: fixing
Parts:
- removed JP7: SolderJumper_3_Open, Jumper:SolderJumper-3_P1.3mm_Open_RoundedPad1.0x1.5mm, symbol Jumper:SolderJumper_3_Open
Connections:
- net CS_IMU2: now also U6.8 (D7/GPIO44)
- net PWM_HAP1: no longer names the net of U6.7 (D6/GPIO43)
Changed lines of the file:
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@@
 	(wire
 		(pts
-			(xy 149.86 73.66) (xy 171.45 73.66)
+			(xy 149.86 73.66) (xy 156.21 73.66)
 		)
 		(stroke
@@
 	(wire
 		(pts
-			(xy 175.26 66.04) (xy 175.26 68.58)
-		)
-		(stroke
-			(width 0)
-			(type default)
-		)
-	)
-	(wire
-		(pts
 			(xy 154.94 83.82) (xy 156.21 83.82)
 		)
@@
 	(wire
 		(pts
-			(xy 177.8 66.04) (xy 175.26 66.04)
-		)
-		(stroke
-			(width 0)
-			(type default)
-		)
-	)
-	(wire
-		(pts
 			(xy 86.36 71.12) (xy 86.36 69.85)
 		)
@@
 	(wire
 		(pts
-			(xy 177.8 81.28) (xy 175.26 81.28)
-		)
-		(stroke
-			(width 0)
-			(type default)
-		)
-	)
-	(wire
-		(pts
 			(xy 153.67 60.96) (xy 153.67 63.5)
 		)
@@
 		(pts
 			(xy 152.4 91.44) (xy 152.4 88.9)
-		)
-		(stroke
-			(width 0)
-			(type default)
-		)
-	)
-	(wire
-		(pts
-			(xy 175.26 81.28) (xy 175.26 78.74)
 		)
 		(stroke
@@
 	(global_label "CS_IMU2"
 		(shape input)
-		(at 177.8 66.04 0)
+		(at 156.21 73.66 0)
 		(fields_autoplaced yes)
 		(effects
@@
 		)
 		(property "Intersheetrefs" "${INTERSHEET_REFS}"
-			(at 188.8285 66.04 0)
+			(at 167.2385 73.66 0)
 			(hide yes)
 			(show_name no)
@@
 		)
 	)
-	(global_label "PWM_HAP2"
-		(shape input)
-		(at 177.8 81.28 0)
-		(fields_autoplaced yes)
-		(effects
-			(font
-				(size 1.27 1.27)
-			)
-			(justify left)
-		)
-		(property "Intersheetrefs" "${INTERSHEET_REFS}"
-			(at 190.8242 81.28 0)
-			(hide yes)
-			(show_name no)
-			(do_not_autoplace no)
-			(effects
-				(font
-					(size 1.27 1.27)
-				)
-				(justify left)
-			)
-		)
-	)
 	(global_label "MOSI"
 		(shape input)
@@
 				)
 				(justify right)
-			)
-		)
-	)
-	(global_label "PWM_HAP1"
-		(shape input)
-		(at 156.21 71.12 0)
-		(fields_autoplaced yes)
-		(effects
-			(font
-				(size 1.27 1.27)
-			)
-			(justify left)
-		)
-		(property "Intersheetrefs" "${INTERSHEET_REFS}"
-			(at 169.2342 71.12 0)
-			(hide yes)
-			(show_name no)
-			(do_not_autoplace no)
-			(effects
-				(font
-					(size 1.27 1.27)
-				)
-				(justify left)
 			)
 		)
@@
 					(unit 1)
 				)
-			)
-		)
-	)
-	(symbol
-		(lib_id "Jumper:SolderJumper_3_Open")
-		(at 175.26 73.66 270)
-		(unit 1)
-		(body_style 1)
-		(exclude_from_sim no)
-		(in_bom no)
-		(on_board yes)
-		(in_pos_files yes)
-		(dnp no)
-		(fields_autoplaced yes)
-		(property "Reference" "JP7"
-			(at 177.8 72.3899 90)
-			(show_name no)
-			(do_not_autoplace no)
-			(effects
-				(font
-					(size 1.27 1.27)
-				)
-				(justify left)
-			)
-		)
-		(property "Value" "SolderJumper_3_Open"
-			(at 177.8 74.9299 90)
-			(show_name no)
-			(do_not_autoplace no)
-			(effects
-				(font
-					(size 1.27 1.27)
-				)
-				(justify left)
-			)
-		)
-		(property "Footprint" "Jumper:SolderJumper-3_P1.3mm_Open_RoundedPad1.0x1.5mm"
-			(at 175.26 73.66 0)
-			(hide yes)
-			(show_name no)
-			(do_not_autoplace no)
-			(effects
-				(font
-					(size 1.27 1.27)
-				)
-			)
-		)
-		(property "Datasheet" ""
-			(at 160.02 73.66 0)
-			(hide yes)
-			(show_name no)
-			(do_not_autoplace no)
-			(effects
-				(font
-					(size 1.27 1.27)
-				)
-			)
-		)
-		(property "Description" "Solder Jumper, 3-pole, open"
-			(at 162.56 73.66 0)
-			(hide yes)
-			(show_name no)
-			(do_not_autoplace no)
-			(effects
-				(font
-					(size 1.27 1.27)
-				)
-			)
-		)
-		(property private "KLC_S5.1" "This is a generic symbol, it has fp-filter, but no default footprint"
-			(at 157.48 73.66 0)
-			(hide yes)
-			(show_name yes)
-			(do_not_autoplace no)
-			(effects
-				(font
-					(size 1.27 1.27)
-				)
-			)
-		)
-		(property private "KLC_S3.3" "Graphical-Symbol: thickness is 6mm, fill is background"
-			(at 154.94 73.66 0)
-			(hide yes)
-			(show_name yes)
-			(do_not_autoplace no)
-			(effects
-				(font
-					(size 1.27 1.27)
-				)
-			)
-		)
-		(pin "1"
-		)
-		(pin "2"
-		)
-		(pin "3"
-		)
-		(instances
-			(project "rehabsense-main"
-				(path "/b751250a-7d43-475a-8447-686d399cd67b/4c292b8e-bacf-4862-ad93-06ae5fddd327"
-					(reference "JP7")
-					(unit 1)
-				)
